File: KiCad/xt-cf.kicad_sch (KiCad schematic)
At the start: 11 parts, among them P1 CF_CARD, U1 PAL20L8, U2 27C128

Commit message: Some touchups, gerbers that were sent to JLPCB ver 0.2
Parts:
- added H1, H2: MountingHole_Pad, MountingHole:MountingHole_3.2mm_M3_ISO7380_Pad, symbol Mechanical:MountingHole_Pad
- C1: value C -> 100n
- C2: value CP1 -> 10u
- R1: value R -> 470
- R2: value R -> 10k
- R3: value R -> 1k
- R4: value R -> 5k6
Connections:
- net GND: now also H1.1, H2.1
