File: KiCad/xt-cf.kicad_pcb (KiCad board)
At the start: 2 copper layers, 99.7 x 71.1 mm, 11 parts, among them P1 CF_CARD, U1 PAL20L8, U2 27C128

Commit message: Some touchups, gerbers that were sent to JLPCB ver 0.2
Parts:
- added H1: MountingHole_Pad, MountingHole:MountingHole_3.2mm_M3_ISO7380_Pad, F.Cu at (190.5, 67.8)
- added H2: MountingHole_Pad, MountingHole:MountingHole_3.2mm_M3_ISO7380_Pad, F.Cu at (190.5, 123.0)
- C1: value C -> 100n
- C2: value CP1 -> 10u
- R1: value R -> 470
- R2: value R -> 10k
- R3: value R -> 1k
- R4: value R -> 5k6
Routing:
- net GND: track 361.8 -> 411.9 mm
- net VCC: track 267.0 -> 271.3 mm
Other:
- board text added: "XT-CF-Pico Version 0.2 Copyright (C) 2025 YO5PTD"
- board text removed: "+"
- board text removed: "20V8"
- board text removed: "27C128"
- board text removed: "XT-CF-Pico Version 0.1 Copyright (C) 2025 YO5PTD"

Commit message: fixes
Routing:
- net /D0: track 153.7 -> 133.5 mm
- net /D1: track 155.8 -> 136.5 mm
- net GND: track 411.9 -> 424.4 mm
- net /~{CF_DASP}: track 117.7 -> 109.5 mm
- net /A1: track 142.1 -> 134.0 mm
- net /A2: track 143.6 -> 136.7 mm
- net VCC: track 271.3 -> 267.7 mm
- net /A3: track 142.3 -> 141.3 mm
Other:
- board text added: "XT-CF-Pico Version 0.3 Copyright (C) 2025 YO5PTD"
- board text removed: "XT-CF-Pico Version 0.2 Copyright (C) 2025 YO5PTD"
